Commit message: DATN

File: ros2_ws/src/ammr/urdf/ammr_base.xacro (robot description, xacro)
@@ -33,4 +33,11 @@
     </collision>
     </link>
+    <link name="base_footprint">
+    </link>
+    <joint name="base_footprint_joint" type="fixed">
+        <origin xyz="0 0 0" rpy="0 0 0" />
+        <parent link="base_link" />
+        <child link="base_footprint" />
+    </joint>
 <!-- CASTER WHEELS LINK-->
     <!-- FRONT RIGHT CASTER WHEELS-->

File: ros2_ws/src/ammr/urdf/ammr_camera.xacro (robot description, xacro)
@@ -33,8 +33,8 @@
     <joint name="Depth_Camera_Joint" type="fixed">
     <origin
-        xyz="0.469 0.002539 ${frame_ground_offset + 0.3676}"
-        rpy="0 0 0" />
+        xyz="0 -0.05834 0.1825"
+        rpy="0 0 -${pi/2}"/>
     <parent
-        link="base_link" />
+        link="Manipulator_J6_Link_1" />
     <child
         link="Depth_Camera_Link" />
@@ -42,3 +42,10 @@
         xyz="0 0 0" />
     </joint>
+    <link name="camera_link">
+    </link>
+    <joint name="camera_link_joint" type="fixed">
+        <origin xyz="0 0 0" rpy="0 0 0" />
+        <parent link="Depth_Camera_Link"/>
+        <child link="camera_link"/>
+    </joint>
 </robot>

File: ros2_ws/src/ammr_mock_components/description/urdf/ammr_base.xacro (robot description, xacro)
@@ -33,4 +33,11 @@
     </collision>
     </link>
+   <link name="base_footprint">
+   </link>
+   <joint name="base_footprint_joint" type="fixed">
+	<origin xyz="0 0 0" rpy="0 0 0" />
+	<parent link="base_link" />
+	<child link="base_footprint" />
+   </joint>
 <!-- CASTER WHEELS LINK-->
     <!-- FRONT RIGHT CASTER WHEELS-->
