Commit message: DATN

File: ros2_ws/src/ammr/urdf/ammr_manipulator.xacro (robot description, xacro)
@@ -341,10 +341,10 @@
     </joint>
     <joint name="EE_1" type="fixed">
-        <origin xyz="0 0 0.07" rpy="0 0 0" />
+        <origin xyz="0 -0.2 0.1" rpy="0 0 ${pi/2}" />
         <parent link="Manipulator_J6_Link_1" />
         <child link="Manipulator_J6_Link_2" />
     </joint>
     <joint name="EE_R" type="prismatic">
-        <origin xyz="-0.04 -0.02 0.01" rpy="${pi/2} 0 0" />
+        <origin xyz="-0.02 0.04 0.01" rpy="${pi/2} 0 ${-pi/2}" />
         <parent link="Manipulator_J6_Link_2" />
         <child link="Manipulator_J6_Link_EER" />
@@ -356,5 +356,5 @@
     </joint>
     <joint name="EE_L" type="prismatic">
-        <origin xyz="0.04 -0.02 0.01" rpy="${-pi/2} 0 ${pi}" />
+        <origin xyz="-0.02 -0.04 0.01" rpy="${-pi/2} 0 ${pi/2}" />
         <parent link="Manipulator_J6_Link_2" />
         <child link="Manipulator_J6_Link_EEL" />
