Commit message: DATN

File: ros2_ws/src/my_robot_hw/description/ros2_control/ammr_main.ros2_control.xacro (robot description, xacro)
@@ -10,4 +10,5 @@
                 <command_interface name="position"/>
                 <command_interface name="velocity"/>
+                <command_interface name="acceleration"/>
                 <state_interface name="position">
                   <param name="initial_value">${initial_positions['Manipulator_J1_Joint']}</param>
@@ -20,4 +21,5 @@
                 <command_interface name="position"/>
                 <command_interface name="velocity"/>
+                <command_interface name="acceleration"/>
                 <state_interface name="position">
                   <param name="initial_value">${initial_positions['Manipulator_J2_Joint']}</param>
@@ -30,4 +32,5 @@
                 <command_interface name="position"/>
                 <command_interface name="velocity"/>
+                <command_interface name="acceleration"/>
                 <state_interface name="position">
                   <param name="initial_value">${initial_positions['Manipulator_J3_Joint']}</param>
@@ -40,4 +43,5 @@
                 <command_interface name="position"/>
                 <command_interface name="velocity"/>
+                <command_interface name="acceleration"/>
                 <state_interface name="position">
                   <param name="initial_value">${initial_positions['Manipulator_J4_Joint']}</param>
@@ -50,4 +54,5 @@
                 <command_interface name="position"/>
                 <command_interface name="velocity"/>
+                <command_interface name="acceleration"/>
                 <state_interface name="position">
                   <param name="initial_value">${initial_positions['Manipulator_J5_Joint']}</param>
@@ -60,4 +65,5 @@
                 <command_interface name="position"/>
                 <command_interface name="velocity"/>
+                <command_interface name="acceleration"/>
                 <state_interface name="position">
                   <param name="initial_value">${initial_positions['Manipulator_J6_Joint']}</param>
@@ -87,4 +93,5 @@
             <joint name="Diff_Wheel_Right_Joint">
                 <command_interface name="velocity"/>
+                <command_interface name="acceleration"/>
                 <state_interface name="position"/>
                 <state_interface name="velocity">
@@ -94,4 +101,5 @@
             <joint name="Diff_Wheel_Left_Joint">
                 <command_interface name="velocity"/>
+                <command_interface name="acceleration"/>
                 <state_interface name="position"/>
                 <state_interface name="velocity">

File: ros2_ws/src/my_robot_hw/description/urdf/ammr_camera.xacro (robot description, xacro)
@@ -33,5 +33,5 @@
     </link>
     <joint name="Depth_Camera_Joint" type="fixed">
-        <origin xyz="-0.058 -0.0025 0.19025" rpy="0 0 -${pi}" />
+        <origin xyz="-0.058 -0.0025 0.19025" rpy="${pi/2} ${pi} -${pi/2}" />
         <parent link="Manipulator_J6_Link" />
         <child link="Depth_Camera_Link" />
@@ -43,5 +43,5 @@
         <parent link="Depth_Camera_Link" />
         <child link="camera_link" />
-        <origin xyz="0 0 0" rpy="0 0 0" />
+        <origin xyz="0 0 0" rpy="${pi/2} -${pi/2} 0" />
     </joint>
 </robot>
